File: Pip Boy wiring/Pip Boy wiring.kicad_sch (KiCad schematic)
At the start: 4 parts, among them J1 GPS Module, J2 MAX10302 Pulse Oximeter, J3 Power Boost

Commit message: Partially completed keyboard in tui, added encoders to wiring diagram
Parts:
- added SW1, SW2, SW3, SW4, SW5: RotaryEncoder, symbol Device:RotaryEncoder
Connections:
- net ENCODER1_A: now reaches U1.11 (GPIO17)
- net ENCODER1_A: now also SW1.A
- net ENCODER1_B: now reaches U1.13 (GPIO27)
- net ENCODER1_B: now also SW1.B
- net ENCODER2_A: now reaches U1.16 (GPIO23)
- net ENCODER2_A: now also SW2.A
- net ENCODER2_B: now reaches U1.18 (GPIO24)
- net ENCODER2_B: now also SW2.B
- net ENCODER3_A: now reaches U1.29 (GPIO5)
- net ENCODER3_A: now also SW3.A
- net ENCODER3_B: now reaches U1.31 (GPIO6)
- net ENCODER3_B: now also SW3.B
- net ENCODER4_A: now reaches U1.35 (GPIO19)
- net ENCODER4_A: now also SW4.A
- net ENCODER4_B: now reaches U1.37 (GPIO26)
- net ENCODER4_B: now also SW4.B
- net ENCODER5_A: now reaches U1.38 (GPIO20)
- net ENCODER5_A: now also SW5.A
- net ENCODER5_B: now reaches U1.40 (GPIO21)
- net ENCODER5_B: now also SW5.B
- net GPS_GND renamed ENCODER_GND
- net ENCODER_GND: now also SW1.C, SW2.C, SW3.C, SW4.C, SW5.C
